Commit message: feat(description): add 3-tier Kachaka shelf macro
_shelf_3tier.urdf.xacro provides a parameterized 3-tier shelf macro
intended to be attached to docking_link so the shelf follows the lift
mechanism. Default dimensions are approximate and can be overridden by
passing depth/width/height/board_thickness/post_size to the macro.

Existing kachaka.urdf.xacro output is unchanged structurally (link and
joint counts identical); only two new shelf materials are added to
_materials.urdf.xacro.

File: ros2/kachaka_description/urdf/_materials.urdf.xacro (robot description, xacro)
@@ -10,3 +10,9 @@
     <color rgba="0.0 0.0 0.0 1.0" />
   </material>
+  <material name="shelf_board">
+    <color rgba="0.85 0.78 0.65 1.0" />
+  </material>
+  <material name="shelf_post">
+    <color rgba="0.15 0.15 0.15 1.0" />
+  </material>
 </robot>
