Commit message: Address Copilot PR review: shelf placement, footprint, dependencies
Five issues raised in PR #3 review (all valid):

1. shelf attached at docking_link with zero offset placed the shelf bottom
   at base_link origin, ~10.75 cm below the real solenoid top. Extend the
   shelf_3tier macro with an `*origin` block and pass z=0.115 m in
   kachaka_with_shelf so shelf_base_link sits on the solenoid top
   (cylinder center 0.1075 + half length 0.0075). Verified offline:
   base_footprint -> os1_lidar z = 0.651 m (was 0.536 m).

2. & 5. Specs/plans documenting the same wrong z value (~0.50 / ~0.61)
   updated to match the corrected URDF (0.615 m for os1_sensor, 0.651 m
   for os1_lidar). TF section in the spec now describes the docking_link
   solenoid offset explicitly.

3. vehicle_info footprint overhangs were inconsistent with the Kachaka
   body collision box. Recompute from _kachaka.urdf.xacro:
     front 0.237, rear 0.150, left 0.120, right 0.120
   Comment in the yaml records the derivation.

4. robot_description.launch.py optionally starts joint_state_publisher,
   so add it as exec_depend in package.xml; documented in the plan too.

xacro expansion still produces 22 links / 21 joints; both packages build
cleanly.

File: ros2/kachaka_autoware_description/urdf/kachaka_with_shelf.urdf.xacro (robot description, xacro)
@@ -12,8 +12,13 @@
   <!--
     docking_link is Kachaka's docking lift mechanism (prismatic joint).
-    Attaching the shelf here makes it follow the lift (up to ~0.012 m),
-    matching real hardware behavior.
+    The frame itself sits at base_link origin; the solenoid that supports
+    the shelf reaches up to z ≈ 0.115 m (cylinder center 0.1075 + half
+    length 0.0075). Mount the shelf bottom there so the published TF
+    matches the physical sensor pose. The shelf still follows the lift
+    (up to +0.012 m) because docking_link is a prismatic child of base_link.
   -->
-  <xacro:shelf_3tier parent="docking_link"/>
+  <xacro:shelf_3tier parent="docking_link">
+    <origin xyz="0 0 0.115" rpy="0 0 0"/>
+  </xacro:shelf_3tier>
   <!-- Mount the Ouster OS-1 at the shelf top center; override origin with values measured in M0 Task 4. -->
   <xacro:ouster_os1 parent="shelf_top">

File: ros2/kachaka_description/urdf/_shelf_3tier.urdf.xacro (robot description, xacro)
@@ -9,4 +9,5 @@
   <xacro:macro name="shelf_3tier"
                params="parent
+                       *origin
                        shelf_name:=shelf
                        depth:=0.32
@@ -19,5 +20,5 @@
       <parent link="${parent}"/>
       <child link="${shelf_name}_base_link"/>
-      <origin xyz="0 0 0" rpy="0 0 0"/>
+      <xacro:insert_block name="origin"/>
     </joint>
     <xacro:macro name="_shelf_board" params="board_name z">
